File: pcbs/minsync/RP2040_minimal_r2.kicad_sch (KiCad schematic)
At the start: 39 parts, among them J1 Comm, J2 Comm, J3 Comm, J4 Comm, J5 SWD_CONN, J6 Conn_01x01_Pin, J7 SSD1306, SW1 SW_Push, U1 NCP1117-3.3_SOT223, U2 W25Q128JVS, U3 RP2040, U4 Si5351A-B-GT, Y2 Crystal_GND24

Commit message: Update TODO
Other:
- note added: "TODO: x check BOOTSEL button: compare to RPi Pico x check if screen would actually fit x check RUN pin with rp minimal change LED in BOM to a better color (C2290?) fix tiny trace error to the right of rp2040"
- note removed: "TODO: x check BOOTSEL button: compare to RPi Pico check if screen would actually fit x check RUN pin with rp minimal"
Changed lines of the file:
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@@
 		)
 	)
-	(text "TODO:\nx check BOOTSEL button: compare to RPi Pico\ncheck if screen would actually fit\nx check RUN pin with rp minimal"
+	(text "TODO:\nx check BOOTSEL button: compare to RPi Pico\nx check if screen would actually fit\nx check RUN pin with rp minimal\nchange LED in BOM to a better color (C2290?)\nfix tiny trace error to the right of rp2040"
 		(exclude_from_sim no)
 		(at 146.558 24.13 0)
