File: pcbs/multiprobe/multiprobe.kicad_pcb (KiCad board)
At the start: 2 copper layers, 50 x 63 mm, 26 parts, among them J1 Display, J10 SWD, J11 SWD, J12 SWD, J13 SWD, J14 SWD, J15 SWD, J16 SWD, J17 SWD, J18 SWD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

Commit message: Order multiprobe v0.1
Changed lines of the file:
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@@
 			(drillshape 0)
 			(scaleselection 1)
-			(outputdirectory "gerber/")
+			(outputdirectory "gerbers")
 		)
 	)
@@
 		)
 		(fp_text user "${REFERENCE}"
-			(at 0 3.81 360)
+			(at 0 3.81 0)
 			(layer "F.Fab")
 			(effects
@@
 	)
 	(segment
-		(start 124 80)
-		(end 120 80)
+		(start 117.46 85.54)
+		(end 118.5 84.5)
 		(width 0.2)
 		(layer "B.Cu")
@@
 	)
 	(segment
-		(start 117.46 77.46)
-		(end 117.46 75.9)
+		(start 117.46 86)
+		(end 117.46 85.54)
 		(width 0.2)
 		(layer "B.Cu")
@@
 	)
 	(segment
-		(start 117.46 86)
-		(end 117.39 85.93)
+		(start 117.46 77.46)
+		(end 117.46 75.9)
 		(width 0.2)
 		(layer "B.Cu")
@@
 	)
 	(segment
-		(start 117.46 86)
-		(end 117.46 85.54)
+		(start 120 80)
+		(end 117.46 77.46)
 		(width 0.2)
 		(layer "B.Cu")
@@
 	)
 	(segment
-		(start 117.39 75.97)
-		(end 117.46 75.9)
+		(start 123.5 84.5)
+		(end 125 83)
 		(width 0.2)
 		(layer "B.Cu")
@@
 	)
 	(segment
-		(start 124 84)
-		(end 125 83)
+		(start 117.46 86)
+		(end 117.39 85.93)
 		(width 0.2)
 		(layer "B.Cu")
@@
 	)
 	(segment
-		(start 125 81)
-		(end 124 80)
+		(start 125 83)
+		(end 125 81)
 		(width 0.2)
 		(layer "B.Cu")
@@
 	)
 	(segment
-		(start 125 83)
-		(end 125 81)
+		(start 124 80)
+		(end 120 80)
 		(width 0.2)
 		(layer "B.Cu")
@@
 	)
 	(segment
-		(start 120 80)
-		(end 117.46 77.46)
+		(start 118.5 84.5)
+		(end 123.5 84.5)
 		(width 0.2)
 		(layer "B.Cu")
@@
 	)
 	(segment
-		(start 117.46 85.54)
-		(end 119 84)
+		(start 117.39 75.97)
+		(end 117.46 75.9)
 		(width 0.2)
 		(layer "B.Cu")
@@
 	)
 	(segment
-		(start 119 84)
-		(end 124 84)
+		(start 125 81)
+		(end 124 80)
 		(width 0.2)
 		(layer "B.Cu")
